Commit message: nav_lecture: add_lecture

File: nav_lecture/xacro/dtw_robot.xacro (robot description, xacro)
@@ -6,4 +6,5 @@
   <xacro:include filename="$(find nav_lecture)/xacro/imu_macro.xacro" />
   <xacro:include filename="$(find nav_lecture)/xacro/camera_macro.xacro" />
+  <xacro:include filename="$(find nav_lecture)/xacro/sonar_macro.xacro" />
   <link name="base_link"/>
   <xacro:body_macro parent="base_link" />
@@ -13,4 +14,5 @@
   <xacro:imu_macro prefix="imu" parent="base_link" xyz="-0.05 0 0.10" robot_name="$(arg robot_name)"/>
   <xacro:camera_macro prefix="head_camera" parent="base_link" xyz="0.1 0 0.08"/>
+  <xacro:sonar_macro prefix="sonar_back" parent="base_link" xyz="-0.2 0 0.08" rpy="0 0 3.1415" robot_name="$(arg robot_name)"/>
   <gazebo>
     <plugin name="gazebo_ros_control" filename="libgazebo_ros_control.so">

File: nav_lecture/xacro/laser_macro.xacro (robot description, xacro)
@@ -33,6 +33,6 @@
               <samples>400</samples>
               <resolution>1</resolution>
-              <min_angle>${radians(-180)}</min_angle>
-              <max_angle>${radians( 180)}</max_angle>
+              <min_angle>${radians(-150)}</min_angle>
+              <max_angle>${radians( 150)}</max_angle>
             </horizontal>
           </scan>

File: nav_lecture/xacro/move_macro.xacro (robot description, xacro)
@@ -13,5 +13,5 @@
       <child  link="${prefix}_link"/>
       <axis xyz="0 0 1" />
-      <limit velocity="12.0" effort="0.4" />
+      <limit velocity="24.0" effort="0.4" />
       <dynamics damping="0.1"/>
     </joint>
